Commit message: feat: gazebo ros bridge

File: ros2_ws/src/my_robot_description/urdf/my_robot.urdf.xacro (robot description, xacro)
@@ -3,3 +3,4 @@
     <xacro:include filename="common_properties.xacro"/>
     <xacro:include filename="robot_base.xacro"/>
+    <xacro:include filename="robot_base_gazebo.xacro"/>
 </robot>

File: ros2_ws/src/my_robot_description/urdf/robot_base.xacro (robot description, xacro)
@@ -1,2 +1,3 @@
+<?xml version="1.0"?>
 <robot xmlns:xacro="http://www.ros.org/wiki/xacro">
     <xacro:property name="base_length" value="0.6"/>
@@ -17,4 +18,10 @@
             <material name="blue"/>
         </visual>
+        <collision>
+            <geometry>
+                <box size="${base_length} ${base_width} ${base_height}"/>
+            </geometry>
+            <origin xyz="0 0 ${base_height / 2.0}" rpy="0 0 0"/>
+        </collision>
         <xacro:box_inertia mass="${robot_weight}" x="${base_length}" y="${base_width}" z="${base_height}"
                             o_xyz="0 0 ${base_height / 2.0}" o_rpy="0 0 0"/>
@@ -29,4 +36,10 @@
                 <material name="black"/>
             </visual>
+            <collision>
+                <geometry>
+                    <sphere radius="${wheel_radius}"/>
+                </geometry>
+                <origin xyz="0 0 0" rpy="0 0 0"/>
+            </collision>
             <xacro:cylinder_inertia mass="${wheel_weight}" radius="${wheel_radius}" height="${wheel_width}"
                                     o_xyz="0 0 0" o_rpy="${pi / 2.0} 0 0"/>
@@ -43,4 +56,10 @@
             <material name="black"/>
         </visual>
+        <collision>
+            <geometry>
+                <sphere radius="${wheel_radius / 2.0}"/>
+            </geometry>
+            <origin xyz="0 0 0" rpy="0 0 0"/>
+        </collision>
         <xacro:sphere_inertia mass="${caster_wheel_weight}" radius="${wheel_radius / 2.0}"
                                 o_xyz="0 0 0" o_rpy="0 0 0"/>
